File: RTSpeed-KiCad/Medio-Puente.kicad_sch (KiCad schematic)
At the start: 30 parts, among them J9 -, Q2 IRFB4321, Q3 IRFB4321, U5 IR2103, U6 INA826

Commit message: PCB redesign (not final)
Parts:
- added C2, C7: 100n, Capacitor_SMD:C_0603_1608Metric, symbol Device:C
- added H1, H2, H3, H4: M3, MountingHole:MountingHole_3.2mm_M3, symbol Mechanical:MountingHole_Pad
- added J1: DATA, Connector_JST:JST_PH_B6B-PH-K_1x06_P2.00mm_Vertical, symbol Connector_Generic:Conn_01x06
- added J2: 12V IN, Connector_JST:JST_PH_B2B-PH-K_1x02_P2.00mm_Vertical, symbol Connector_Generic:Conn_01x02
- added J4: +24V IN, MountingHole:MountingHole_2.5mm_Pad_TopBottom, symbol Connector:Screw_Terminal_01x01
- added J5: GND IN, MountingHole:MountingHole_2.5mm_Pad_TopBottom, symbol Connector:Screw_Terminal_01x01
- added J6: TEMP, Connector_JST:JST_PH_B3B-PH-K_1x03_P2.00mm_Vertical, symbol Connector_Generic:Conn_01x03
- added R11, R5: 22R, Resistor_SMD:R_0603_1608Metric, symbol Device:R_US
- added R3, R8: 10k 1%, Resistor_SMD:R_0603_1608Metric, symbol Device:R_US
- added TH1, TH2: 10k, RTSpeed:temp sensor, symbol Device:Thermistor_NTC
- renumbered C21 to C1, C28 to C10, C29 to C11, C30 to C12, C22 to C3, C23 to C4, C24 to C5, C25 to C6, C26 to C8, C27 to C9, D20 to D1, D21 to D2, D22 to D3, D23 to D4, J9 to J3, Q2 to Q1, Q3 to Q2, R27 to R1, R33 to R10, R34 to R12, R35 to R13, R36 to R14, R37 to R15, R28 to R2, R29 to R4, R30 to R6, R31 to R7, R32 to R9, U5 to U1, U6 to U2
Connections:
- net +12V: now also J2.2 (Pin_2)
- net +24V: now also J4.1 (Pin_1)
- net +3V3: now also J1.6 (Pin_6), R3.2, R8.2
- net GND: now also C2.2, C7.2, J1.1 (Pin_1), J2.1 (Pin_1), J5.1 (Pin_1), J6.1 (Pin_1), TH1.2, TH2.2
- net HIN: now also J1.2 (Pin_2)
- net I_SENSE: now also J1.4 (Pin_4)
- net NLIN: now also J1.3 (Pin_3)
- net V_SENSE: now also J1.5 (Pin_5)
- net PHASE_OUT renamed OUT
- new net: C7.1, R11.2, R8.1, TH2.1
- new net: C2.1, R3.1, R5.2, TH1.1
- new net TH: J6.2 (Pin_2), R5.1
- new net TL: J6.3 (Pin_3), R11.1
- no-connect marks 0 -> 4
Other:
- note added: "Sensores de temperatura (1 por MOSFET)"
- note added: "Tornillos"
- moved on the sheet: C10, C12, C4, C5, C8, D1, D2, D4, R1, R14, R15, R2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
