File: RTSpeed-KiCad/RTSpeed-KiCad.kicad_pcb (KiCad board)
At the start: 4 copper layers, 155 x 116 mm, 228 parts, among them J1 24V IN, J10 -, J11 -, J12 I^{2}C, J13 24V DC, J14 230V AC, J15 Contactor Coil, J2 USB C Receptacle, J3 MOTOR, J4 -, J5 -, J6 -, J7 SWD-I^{2}C, J8 SENSORES HALL, J9 -, K1 Relay 24VDC, Q1 DMG3402L, Q2 IRFB4321, Q3 IRFB4321, Q4 IRFB4321, Q5 IRFB4321, Q6 IRFB4321, Q7 IRFB4321, Q8 2N2222, Q9 IRFB4321, SW1 BOOT0, SW2 NRST, U1 STM32F411CEUx, U10 INA826, U11 ATtiny85-20P, U2 LM317L, U3 ADS7830, U4 LM317, U5 IR2103, U6 INA826, U7 IR2103, U8 INA826, U9 IR2103, Y1 25MHz, Y2 32.768kHz

Commit message: Contactor control pcb
Parts:
- added H5: M3, MountingHole:MountingHole_3.2mm_M3, F.Cu at (83.5, 171.7)
- added H6: M3, MountingHole:MountingHole_3.2mm_M3, F.Cu at (83.5, 139.2)
- added H7: M3, MountingHole:MountingHole_3.2mm_M3, F.Cu at (156.2, 139.2)
- added H9: M3, MountingHole:MountingHole_3.2mm_M3, F.Cu at (156.2, 171.7)
- added REF**: Symbol_HighVoltage_Triangle_6x6mm_Copper, Symbol:Symbol_HighVoltage_Triangle_6x6mm_Copper, F.Cu at (90.7, 139.2)
- K1: footprint Relay_THT:Relay_SPDT_HsinDa_Y14 -> ESC-TFG-KiCad:OMRON G2R-1
- moved R77 20.0 mm to (118.3, 137.9), turned to 180 degrees
- moved K1 19.1 mm to (126.2, 144.3), turned to 0 degrees
- moved R76 17.1 mm to (103.1, 141.1)
- moved REF** 11.6 mm to (90.4, 171.2)
- moved J15 10.9 mm to (142.5, 167.2)
- moved J14 10.9 mm to (120.2, 167.2)
- moved J13 10.9 mm to (98.0, 167.2)
- moved REF** 10.2 mm to (133.3, 171.2)
- moved REF** 10.2 mm to (145.0, 171.2)
- moved REF** 10.2 mm to (126.0, 171.5)
- moved Q9 9.49 mm to (114.1, 145.8)
- moved D32 6.94 mm to (120.6, 152.2), turned to 90 degrees
- moved U11 6.87 mm to (103.1, 151.9)
- moved J12 6.20 mm to (90.2, 151.9)
- moved Q8 4.91 mm to (108.8, 149.6), turned to 90 degrees
Connections:
- K1 pad 1: /Contactor-Control/Phase -> +24V
- K1 pad 3: Net-(D32-A) -> /Contactor-Control/Phase
- K1 pad 4: +24V -> /Contactor-Control/Cont Ctrl
- K1 pad 5: /Contactor-Control/Cont Ctrl -> Net-(D32-A)
Routing:
- net /Contactor-Control/Phase: track 52.4 -> 39.0 mm
- net +24V: track 189.0 -> 177.8 mm
- net Net-(Q8-C): track 12.4 -> 22.3 mm
- net Net-(D32-A): track 21.8 -> 13.8 mm
- net Net-(U11-PB1): track 16.8 -> 10.00 mm
- net Net-(Q8-B): track 8.93 -> 15.5 mm
- net /Contactor-Control/SCL: track 4.86 -> 6.33 mm
- net +3V3: track 361.6 -> 363.1 mm
- net /Contactor-Control/Cont Ctrl: track 18.5 -> 19.5 mm
- net /Contactor-Control/SDA: track 6.66 -> 7.36 mm
- net GND: vias 625 -> 751
- net (no net): vias 0 -> 2
Other:
- board size 155 x 116 mm -> 155 x 111.3 mm

Commit message: PCB redesign (not final)
Parts:
- removed D32: 1N4148, Diode_THT:D_DO-35_SOD27_P7.62mm_Horizontal
- removed G***: LOGO, TFG-Brushless-ESC:logo
- removed REF** (x2): Symbol_HighVoltage_Triangle_6x6mm_Copper, Symbol:Symbol_HighVoltage_Triangle_6x6mm_Copper
- removed REF**: OSHW-Logo2_9.8x8mm_SilkScreen, Symbol:OSHW-Logo2_9.8x8mm_SilkScreen
- removed REF**: WEEE-Logo_4.2x6mm_SilkScreen, Symbol:WEEE-Logo_4.2x6mm_SilkScreen
- removed REF**: OSHW-Symbol_6.7x6mm_SilkScreen, Symbol:OSHW-Symbol_6.7x6mm_SilkScreen
- removed REF** (x2): KiCad-Logo2_5mm_SilkScreen, Symbol:KiCad-Logo2_5mm_SilkScreen
- removed U11: ATtiny85-20P, Package_DIP:DIP-8_W7.62mm
- added H10: M3, MountingHole:MountingHole_3.2mm_M3, F.Cu at (190.1, 33.7)
- added H11: M3, MountingHole:MountingHole_3.2mm_M3, F.Cu at (254.1, 53.7)
- added H12: M3, MountingHole:MountingHole_3.2mm_M3, F.Cu at (254.1, 33.7)
- added H13: M3, MountingHole:MountingHole_3.2mm_M3, F.Cu at (110.8, 111.8)
- added H14: M3, MountingHole:MountingHole_3.2mm_M3, F.Cu at (110.8, 75.3)
- added H15: M3, MountingHole:MountingHole_3.2mm_M3, F.Cu at (45.8, 112.0)
- added H16: M3, MountingHole:MountingHole_3.2mm_M3, F.Cu at (45.8, 75.3)
- added H17: M3, MountingHole:MountingHole_3.2mm_M3, F.Cu at (255.1, 110.3)
- added H18: M3, MountingHole:MountingHole_3.2mm_M3, F.Cu at (255.1, 73.8)
- added H19: M3, MountingHole:MountingHole_3.2mm_M3, F.Cu at (70.0, 155.8)
- added H20: M3, MountingHole:MountingHole_3.2mm_M3, F.Cu at (89.9, 155.8)
- added H21: M3, MountingHole:MountingHole_3.2mm_M3, F.Cu at (89.9, 211.7)
- added H22: M3, MountingHole:MountingHole_3.2mm_M3, F.Cu at (70.0, 211.7)
- added H23: M3, MountingHole:MountingHole_3.2mm_M3, F.Cu at (133.3, -29.7)
- added H24: M3, MountingHole:MountingHole_3.2mm_M3, F.Cu at (193.3, -9.68)
- added H25: M3, MountingHole:MountingHole_3.2mm_M3, F.Cu at (193.3, -29.7)
- added H26: M3, MountingHole:MountingHole_3.2mm_M3, F.Cu at (133.3, -9.68)
- added H8: M3, MountingHole:MountingHole_3.2mm_M3, F.Cu at (181.4, 33.7)
- added J16: +24V IN, MountingHole:MountingHole_2.5mm_Pad_TopBottom, F.Cu at (207.1, 48.9)
- added J17: GND IN, MountingHole:MountingHole_2.5mm_Pad_TopBottom, F.Cu at (198.0, 48.9)
- added J18: TEMP, Connector_JST:JST_PH_B3B-PH-K_1x03_P2.00mm_Vertical, F.Cu at (238.1, 53.9)
- added J19: USB C Receptacle, Connector_USB:USB_C_Receptacle_XKB_U262-16XN-4BVC11, F.Cu at (163.3, -7.18)
- added J20: U, Connector_JST:JST_PH_B6B-PH-K_1x06_P2.00mm_Vertical, F.Cu at (139.8, -32.2)
- added J21: V, Connector_JST:JST_PH_B6B-PH-K_1x06_P2.00mm_Vertical, F.Cu at (158.3, -32.2)
- added J22: SWD-I^{2}C, Connector_PinHeader_2.54mm:PinHeader_2x04_P2.54mm_Vertical, F.Cu at (153.7, -9.00)
- added J23: GPIO, Connector_JST:JST_PH_B3B-PH-K_1x03_P2.00mm_Vertical, F.Cu at (130.7, -17.7)
- added J24: W, Connector_JST:JST_PH_B6B-PH-K_1x06_P2.00mm_Vertical, F.Cu at (176.8, -32.2)
- added J25: HALL IN, Connector_JST:JST_PH_B5B-PH-K_1x05_P2.00mm_Vertical, F.Cu at (195.8, -23.7)
- added J26: GPIO, Connector_JST:JST_PH_B2B-PH-K_1x02_P2.00mm_Vertical, F.Cu at (46.4, 102.4)
- added J27: 24V, RTSpeed:Barrier_1x02, F.Cu at (61.3, 107.8)
- added J28: +24V OUT, MountingHole:MountingHole_2.5mm_Pad_TopBottom, F.Cu at (76.8, 179.0)
- added J29: VSENSE, Connector_JST:JST_PH_B3B-PH-K_1x03_P2.00mm_Vertical, F.Cu at (246.0, 78.4)
- added J30: SENSORES HALL, Connector_JST:JST_PH_S5B-PH-K_1x05_P2.00mm_Horizontal, F.Cu at (-40.0, 127.3)
- added J31: HALL OUT, Connector_JST:JST_PH_B5B-PH-K_1x05_P2.00mm_Vertical, F.Cu at (-40.0, 136.9)
- added J32: MOTOR, RTSpeed:Barrier_1x03, F.Cu at (-33.9, 116.2)
- added J33: -, MountingHole:MountingHole_2.5mm_Pad_TopBottom, F.Cu at (-46.2, 128.2)
- added J34: -, MountingHole:MountingHole_2.5mm_Pad_TopBottom, F.Cu at (-46.2, 134.7)
- added J35: -, MountingHole:MountingHole_2.5mm_Pad_TopBottom, F.Cu at (-46.2, 141.3)
- added J36: GND OUT, MountingHole:MountingHole_2.5mm_Pad_TopBottom, F.Cu at (76.8, 185.5)
- added J37: +24V OUT, MountingHole:MountingHole_2.5mm_Pad_TopBottom, F.Cu at (83.4, 179.0)
- added J38: GND OUT, MountingHole:MountingHole_2.5mm_Pad_TopBottom, F.Cu at (83.4, 185.5)
- added J39: +24V OUT, MountingHole:MountingHole_2.5mm_Pad_TopBottom, F.Cu at (89.9, 179.0)
- added J40: GND OUT, MountingHole:MountingHole_2.5mm_Pad_TopBottom, F.Cu at (89.9, 185.5)
- added J41: I^{2}C, Connector_JST:JST_PH_B3B-PH-K_1x03_P2.00mm_Vertical, F.Cu at (182.8, -8.23)
- added J42: I^{2}C, Connector_JST:JST_PH_B3B-PH-K_1x03_P2.00mm_Vertical, F.Cu at (246.0, 107.3)
- added J43: +24V OUT, MountingHole:MountingHole_2.5mm_Pad_TopBottom, F.Cu at (75.8, 104.0)
- added J44: GND OUT, MountingHole:MountingHole_2.5mm_Pad_TopBottom, F.Cu at (75.8, 112.5)
- added J45: +24V IN, MountingHole:MountingHole_2.5mm_Pad_TopBottom, F.Cu at (70.0, 204.9)
- added J46: GND IN, MountingHole:MountingHole_2.5mm_Pad_TopBottom, F.Cu at (78.8, 204.9)
- added J47: 12V IN, Connector_JST:JST_PH_B2B-PH-K_1x02_P2.00mm_Vertical, F.Cu at (88.8, 164.1)
- added J48: SENS, Connector_JST:JST_PH_B3B-PH-K_1x03_P2.00mm_Vertical, F.Cu at (88.8, 173.2)
- added J49: DATA, Connector_JST:JST_PH_B8B-PH-K_1x08_P2.00mm_Vertical, F.Cu at (246.0, 97.9)
- added R78: 10k, Resistor_SMD:R_0603_1608Metric, F.Cu at (-18.6, 131.2)
- C1: value 20p -> 2.2u; footprint Capacitor_SMD:C_0603_1608Metric -> Capacitor_SMD:CP_Elec_4x5.4
- C10, C22, C34: value 100n -> 10p
- C11: value 100n -> 1000u; footprint Capacitor_SMD:C_0603_1608Metric -> Capacitor_THT:CP_Radial_D12.5mm_P5.00mm
- C13, C25: value 10u -> 2.2u
- C14, C19: value 10u -> 100n; footprint Capacitor_SMD:CP_Elec_4x5.4 -> Capacitor_SMD:C_0603_1608Metric
- C16, C32: value 100n -> 1n
- C2: value 15p -> 100n
- C20: value 10u -> 1n; footprint Capacitor_SMD:CP_Elec_4x5.4 -> Capacitor_SMD:C_0603_1608Metric
- C21, C31, C41: value 2.2u -> 100n; footprint Capacitor_SMD:CP_Elec_4x5.4 -> Capacitor_SMD:C_0603_1608Metric
- C23: value 1n -> 1000u; footprint Capacitor_SMD:C_0603_1608Metric -> Capacitor_THT:CP_Radial_D12.5mm_P5.00mm
- C26, C33, C36: value 1n -> 100n
- C28: value 10p -> 1n
- C29: value 1000u -> 100n; footprint Capacitor_THT:CP_Radial_D12.5mm_P5.00mm -> Capacitor_SMD:C_0603_1608Metric
- C30, C40, C50, C55, C56, C6: value 100n -> 10u; footprint Capacitor_SMD:C_0603_1608Metric -> Capacitor_SMD:CP_Elec_4x5.4
- C35: value 10u -> 1000u; footprint Capacitor_SMD:CP_Elec_4x5.4 -> Capacitor_THT:CP_Radial_D12.5mm_P5.00mm
- C38, C48: value 10p -> 100n
- C39: value 1000u -> 10u; footprint Capacitor_THT:CP_Radial_D12.5mm_P5.00mm -> Capacitor_SMD:CP_Elec_4x5.4
- C4: value 15p -> 1n
- C42: value 100n -> 20p
- C43: value 1n -> 15p
- C45: value 10u -> 15p; footprint Capacitor_SMD:CP_Elec_4x5.4 -> Capacitor_SMD:C_0603_1608Metric
- C46: value 1n -> 20p
- C49: value 1000u -> 2u2 X7R Ceramic; footprint Capacitor_THT:CP_Radial_D12.5mm_P5.00mm -> Capacitor_SMD:C_0603_1608Metric
- C5: value 20p -> 100n
- C8: value 2u2 X7R Ceramic -> 1n
- D1, D10, D2, D3: value GREEN -> 1N4148; footprint LED_SMD:LED_0805_2012Metric -> Diode_SMD:D_SOD-123
- D11: value DESD5V0U1BA -> 1N4148; footprint Diode_SMD:D_SOD-323_HandSoldering -> Diode_SMD:D_SOD-123
- D12: value SMBJ28CA -> DESD5V0U1BA; footprint Diode_SMD:D_SMB -> Diode_SMD:D_SOD-323_HandSoldering
- D14: value SMBJ28CA -> STPS40170C; footprint Diode_SMD:D_SMB -> Package_TO_SOT_THT:TO-220-3_Vertical
- D15, D17: value D5V0L2B3T -> GREEN; footprint Package_TO_SOT_SMD:SOT-523 -> LED_SMD:LED_0805_2012Metric
- D16: value D5V0L2B3T -> SD12CT1; footprint Package_TO_SOT_SMD:SOT-523 -> Diode_SMD:D_SOD-323_HandSoldering
- D18: value SD12CT1 -> D5V0L2B3T; footprint Diode_SMD:D_SOD-323_HandSoldering -> Package_TO_SOT_SMD:SOT-523
- D19: value D5V0L2B3T -> DESD5V0U1BA; footprint Package_TO_SOT_SMD:SOT-523 -> Diode_SMD:D_SOD-323_HandSoldering
- D20, D21, D25: value 1N4148 -> GREEN; footprint Diode_SMD:D_SOD-123 -> LED_SMD:LED_0805_2012Metric
- D22, D24, D28: value 1N4148 -> D5V0L2B3T; footprint Diode_SMD:D_SOD-123 -> Package_TO_SOT_SMD:SOT-523
- D26: footprint Diode_SMD:D_SOD-123 -> Diode_THT:D_DO-35_SOD27_P7.62mm_Horizontal
- D27: value DESD5V0U1BA -> D5V0L2B3T; footprint Diode_SMD:D_SOD-323_HandSoldering -> Package_TO_SOT_SMD:SOT-523
- D29, D30: value 1N4148 -> SMBJ28CA; footprint Diode_SMD:D_SOD-123 -> Diode_SMD:D_SMB
- D31: value DESD5V0U1BA -> SMBJ28CA; footprint Diode_SMD:D_SOD-323_HandSoldering -> Diode_SMD:D_SMB
- D4: value GREEN -> DESD5V0U1BA; footprint LED_SMD:LED_0805_2012Metric -> Diode_SMD:D_SOD-323_HandSoldering
- D5: value SMBJ28CA -> 1N4148; footprint Diode_SMD:D_SMB -> Diode_SMD:D_SOD-123
- D6: value STPS40170C -> 1N4148; footprint Package_TO_SOT_THT:TO-220-3_Vertical -> Diode_SMD:D_SOD-123
- D7: value D5V0L2B3T -> 1N4148; footprint Package_TO_SOT_SMD:SOT-523 -> Diode_SMD:D_SOD-123
- D9: value B240A-13-F -> 1N4148; footprint Diode_SMD:D_SMA -> Diode_SMD:D_SOD-123
- F1: footprint TFG-Brushless-ESC:Fuseholder_Automotive -> RTSpeed:Fuseholder_Automotive
- H1, H2, H3, H4: footprint MountingHole:MountingHole_3.2mm_M3_Pad_Via -> MountingHole:MountingHole_3.2mm_M3
- J1: value 24V IN -> DATA; footprint TFG-Brushless-ESC:Barrier_1x02 -> Connector_JST:JST_PH_B6B-PH-K_1x06_P2.00mm_Vertical
- J10, J4: value - -> +24V IN
- J11, J5: value - -> GND IN
- J12: value I^{2}C -> TEMP; footprint Connector_PinHeader_2.54mm:PinHeader_1x04_P2.54mm_Horizontal -> Connector_JST:JST_PH_B3B-PH-K_1x03_P2.00mm_Vertical
- J13: value 24V DC -> DATA; footprint ESC-TFG-KiCad:Barrier_1x02 -> Connector_JST:JST_PH_B6B-PH-K_1x06_P2.00mm_Vertical
- J14: value 230V AC -> 12V IN; footprint ESC-TFG-KiCad:Barrier_1x02 -> Connector_JST:JST_PH_B2B-PH-K_1x02_P2.00mm_Vertical
- J15: value Contactor Coil -> -; footprint ESC-TFG-KiCad:Barrier_1x02 -> MountingHole:MountingHole_2.5mm_Pad_TopBottom
- J2: value USB C Receptacle -> 12V IN; footprint Connector_USB:USB_C_Receptacle_XKB_U262-16XN-4BVC11 -> Connector_JST:JST_PH_B2B-PH-K_1x02_P2.00mm_Vertical
- J3: value MOTOR -> -; footprint TFG-Brushless-ESC:Barrier_1x03 -> MountingHole:MountingHole_2.5mm_Pad_TopBottom
- J6: value - -> TEMP; footprint MountingHole:MountingHole_2.5mm_Pad_TopBottom -> Connector_JST:JST_PH_B3B-PH-K_1x03_P2.00mm_Vertical
- J7: value SWD-I^{2}C -> DATA; footprint Connector_PinHeader_2.54mm:PinHeader_2x04_P2.54mm_Horizontal -> Connector_JST:JST_PH_B6B-PH-K_1x06_P2.00mm_Vertical
- J8: value SENSORES HALL -> 12V IN; footprint Connector_JST:JST_PH_S5B-PH-K_1x05_P2.00mm_Horizontal -> Connector_JST:JST_PH_B2B-PH-K_1x02_P2.00mm_Vertical
- K1: footprint ESC-TFG-KiCad:OMRON G2R-1 -> Relay_THT:Relay_SPDT_RAYEX-L90
- Q1: value DMG3402L -> IRFB4321; footprint Package_TO_SOT_SMD:SOT-23 -> Package_TO_SOT_THT:TO-220-3_Vertical
- Q7: value IRFB4321 -> DMG3402L; footprint Package_TO_SOT_THT:TO-220-3_Vertical -> Package_TO_SOT_SMD:SOT-23
- Q8: footprint Package_TO_SOT_THT:TO-92 -> Package_TO_SOT_THT:TO-92_Inline
- R1, R16: value 1k -> 2mR 1%; footprint Resistor_SMD:R_0603_1608Metric -> Resistor_SMD:R_2512_6332Metric
- R10: value 22R -> 10R; footprint Resistor_SMD:R_0603_1608Metric -> Resistor_SMD:R_0805_2012Metric
- R12, R43, R54: value 10R -> 10k; footprint Resistor_SMD:R_0805_2012Metric -> Resistor_SMD:R_0603_1608Metric
- R14: value 390R 1% -> 10k 1%
- R15: value 1k -> 1k 1%
- R17: value 240R 1% -> 330R
- R19: value 390R 1% -> 1k5
- R2: value 1k -> 330R
- R20: value 390R 1% -> 22R
- R21, R6: value 10k -> 330R
- R22: value 390R 1% -> 10k
- R23, R3: value 10k -> 10k 1%
- R24, R25: value 10k -> 10R; footprint Resistor_SMD:R_0603_1608Metric -> Resistor_SMD:R_0805_2012Metric
- R26, R35, R5: value 10k -> 22R
- R27: value 2mR 1% -> 10k; footprint Resistor_SMD:R_2512_6332Metric -> Resistor_SMD:R_0603_1608Metric
- R28: value 330R -> 10k
- R29: value 1k5 -> 10k 1%
- R30: value 330R -> 1k 1%
- R31: value 10k -> 2mR 1%; footprint Resistor_SMD:R_0603_1608Metric -> Resistor_SMD:R_2512_6332Metric
- R32: value 10R -> 330R; footprint Resistor_SMD:R_0805_2012Metric -> Resistor_SMD:R_0603_1608Metric
- R33, R44: value 10R -> 10k 1%; footprint Resistor_SMD:R_0805_2012Metric -> Resistor_SMD:R_0603_1608Metric
- R34, R4: value 10k -> 1k5
- R36: value 10k 1% -> 330R
- R37: value 1k 1% -> 10k
- R38, R49: value 2mR 1% -> 10k 1%; footprint Resistor_SMD:R_2512_6332Metric -> Resistor_SMD:R_0603_1608Metric
- R39: value 330R -> 10R; footprint Resistor_SMD:R_0603_1608Metric -> Resistor_SMD:R_0805_2012Metric
- R40: value 1k5 -> 10R; footprint Resistor_SMD:R_0603_1608Metric -> Resistor_SMD:R_0805_2012Metric
- R41: value 330R -> 22R
- R45: value 10k -> 1k 1%
- R50, R52: value 330R -> 390R 1%
- R51: value 1k5 -> 390R 1%
- R55: value 10R -> 1k 1%; footprint Resistor_SMD:R_0805_2012Metric -> Resistor_SMD:R_0603_1608Metric
- R56: value 10k -> 240R 1%
- R58, R68: value 10k 1% -> 10k
- R59: value 1k 1% -> 22R
- R60: value 10k 1% -> 22R
- R61, R62: value 10k 1% -> 5k1
- R63, R64, R65: value 22R -> 1k
- R66: value 10k 1% -> 10R; footprint Resistor_SMD:R_0603_1608Metric -> Resistor_SMD:R_0805_2012Metric
- R67: value 10k 1% -> 390R 1%
- R69: value 22R -> 240R 1%
- R70, R71: value 22R -> 5k1
- R72: value 1k 1% -> 1k
- R73: value 10k 1% -> 1k; footprint Resistor_SMD:R_0603_1608Metric -> Resistor_THT:R_Axial_DIN0207_L6.3mm_D2.5mm_P15.24mm_Horizontal
- R74: value 240R 1% -> 10k; footprint Resistor_SMD:R_0603_1608Metric -> Resistor_THT:R_Axial_DIN0207_L6.3mm_D2.5mm_P15.24mm_Horizontal
- R75: value 1k 1% -> 100R 10W; footprint Resistor_SMD:R_0603_1608Metric -> RTSpeed:R_Power_22x9.5x9.5_P18mm
- R76: value 1k -> 10k; footprint Resistor_THT:R_Axial_DIN0207_L6.3mm_D2.5mm_P15.24mm_Horizontal -> Resistor_SMD:R_0603_1608Metric
- R77: footprint Resistor_THT:R_Axial_DIN0207_L6.3mm_D2.5mm_P15.24mm_Horizontal -> Resistor_SMD:R_0603_1608Metric
- R8: value 5k1 -> 10k 1%
- R9: value 5k1 -> 10R; footprint Resistor_SMD:R_0603_1608Metric -> Resistor_SMD:R_0805_2012Metric
- TH1, TH2, TH3, TH4, TH5, TH6: footprint TFG-Brushless-ESC:temp sensor -> RTSpeed:temp sensor
- U1: value STM32F411CEUx -> IR2103; footprint Package_DFN_QFN:QFN-48-1EP_7x7mm_P0.5mm_EP5.6x5.6mm -> Package_SO:SOIC-8_3.9x4.9mm_P1.27mm
- U10: value INA826 -> ADS7830; footprint Package_SO:SOIC-8_3.9x4.9mm_P1.27mm -> Package_SO:TSSOP-16_4.4x5mm_P0.65mm
- U2: value LM317L -> INA826; footprint Package_TO_SOT_SMD:SOT-89-3 -> Package_SO:SOIC-8_3.9x4.9mm_P1.27mm
- U3: value ADS7830 -> IR2103; footprint Package_SO:TSSOP-16_4.4x5mm_P0.65mm -> Package_SO:SOIC-8_3.9x4.9mm_P1.27mm
- U4: value LM317 -> INA826; footprint Package_TO_SOT_THT:TO-220-3_Vertical -> Package_SO:SOIC-8_3.9x4.9mm_P1.27mm
- U7: value IR2103 -> LM317; footprint Package_SO:SOIC-8_3.9x4.9mm_P1.27mm -> Package_TO_SOT_THT:TO-220-3_Vertical
- U8: value INA826 -> STM32F411CEUx; footprint Package_SO:SOIC-8_3.9x4.9mm_P1.27mm -> Package_DFN_QFN:QFN-48-1EP_7x7mm_P0.5mm_EP5.6x5.6mm
- U9: value IR2103 -> LM317L; footprint Package_SO:SOIC-8_3.9x4.9mm_P1.27mm -> Package_TO_SOT_SMD:SOT-89-3
- moved D29 243.0 mm to (-24.8, 127.7), turned to 0 degrees
- moved D31 241.6 mm to (-24.8, 138.8)
- moved D30 222.5 mm to (-24.8, 133.2), turned to 0 degrees
- moved D28 213.4 mm to (-18.7, 137.2), turned to 0 degrees
- moved R5 207.6 mm to (57.0, -32.4)
- moved D27 189.8 mm to (-18.7, 134.0)
- moved D3 184.7 mm to (79.2, -20.5), turned to -90 degrees
- moved J3 182.4 mm to (83.3, -31.2)
- moved J4 180.0 mm to (68.5, -15.8)
- moved J5 179.7 mm to (59.4, -15.8)
- moved H4 178.6 mm to (113.3, -29.7)
- moved R3 175.7 mm to (62.4, -33.2)
- moved R6 175.0 mm to (99.9, -31.2), turned to 90 degrees
- moved C2 170.9 mm to (59.3, -33.2), turned to 180 degrees
- moved J13 168.0 mm to (222.2, 53.9)
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Connections:
- C1 pad 1: /HSE_1 -> +12V
- C10 pad 1: +3V3 -> GND
- C10 pad 2: GND -> /Microcontrolador/PB1
- C11 pad 1: VDDA -> +24V
- C12 pad 1: +5V -> /Microcontrolador/PB0
- C13 pad 1: +5V -> +12V
- C14 pad 1: +3V3 -> Net-(C14-Pad1)
- C15 pad 1: +24V -> +12V
- C16 pad 1: +3V3 -> Net-(D5-K)
- C16 pad 2: GND -> /Medio-Puente-V/PHASE_OUT
- C17 pad 1: Net-(U3-REFin/REFout) -> +3V3
- C18 pad 1: +24V -> /Medio-Puente-V/VB
- C18 pad 2: GND -> /Medio-Puente-V/PHASE_OUT
- C19 pad 1: +3V3 -> Net-(C19-Pad1)
- C2 pad 1: /LSE_1 -> Net-(C2-Pad1)
- C20 pad 1: +12V -> Net-(D6-K)
- C20 pad 2: GND -> /Medio-Puente-V/Shunt
- C21 pad 1: +12V -> /Medio-Puente-V/VB
- C21 pad 2: GND -> /Medio-Puente-V/PHASE_OUT
- C22 pad 1: +12V -> GND
- C22 pad 2: GND -> /Microcontrolador/PA5
- C23 pad 1: Net-(D20-K) -> +24V
- C23 pad 2: /Medio-Puente-U/PHASE_OUT -> GND
- C24 pad 1: +3V3 -> /Microcontrolador/PA4
- C25 pad 1: /Medio-Puente-U/VB -> +12V
- C25 pad 2: /Medio-Puente-U/PHASE_OUT -> GND
- C26 pad 1: Net-(D21-K) -> Net-(C26-Pad1)
- C26 pad 2: /Medio-Puente-U/Shunt -> GND
- C27 pad 1: /Medio-Puente-U/VB -> +12V
- C27 pad 2: /Medio-Puente-U/PHASE_OUT -> GND
- C28 pad 1: GND -> Net-(D9-K)
- C28 pad 2: /PB0 -> /Medio-Puente-W/PHASE_OUT
- C29 pad 1: +24V -> +3V3
- C3 pad 1: GND -> +12V
- C3 pad 2: /NRST -> GND
- C30 pad 1: /PB1 -> /Medio-Puente-W/VB
- C30 pad 2: GND -> /Medio-Puente-W/PHASE_OUT
- C31 pad 1: +12V -> Net-(C31-Pad1)
- C32 pad 1: +12V -> Net-(D10-K)
- C32 pad 2: GND -> /Medio-Puente-W/Shunt
- C33 pad 1: Net-(D24-K) -> /Medio-Puente-W/VB
- C33 pad 2: /Medio-Puente-V/PHASE_OUT -> /Medio-Puente-W/PHASE_OUT
- C34 pad 1: +3V3 -> GND
- C34 pad 2: GND -> /Microcontrolador/PA1
- C35 pad 1: /Medio-Puente-V/VB -> +24V
- C35 pad 2: /Medio-Puente-V/PHASE_OUT -> GND
- C36 pad 1: Net-(D25-K) -> /Microcontrolador/PA0
- C36 pad 2: /Medio-Puente-V/Shunt -> GND
- C37 pad 1: /Medio-Puente-V/VB -> /ADC/CH0
- C37 pad 2: /Medio-Puente-V/PHASE_OUT -> GND
- C38 pad 1: GND -> +24V
- C38 pad 2: /PA4 -> GND
- C4 pad 1: /LSE_2 -> Net-(D1-K)
- C4 pad 2: GND -> /Medio-Puente-U/PHASE_OUT
- C40 pad 1: /PA5 -> +12V
- C41 pad 1: +12V -> /ADC/CH1
- C42 pad 1: +12V -> /Microcontrolador/HSE_1
- C43 pad 1: Net-(D28-K) -> /Microcontrolador/LSE_1
- C43 pad 2: /Medio-Puente-W/PHASE_OUT -> GND
- C44 pad 1: +3V3 -> GND
- C44 pad 2: GND -> /Microcontrolador/NRST
- C45 pad 1: /Medio-Puente-W/VB -> /Microcontrolador/LSE_2
- C45 pad 2: /Medio-Puente-W/PHASE_OUT -> GND
- C46 pad 1: Net-(D29-K) -> /Microcontrolador/HSE_2
- C46 pad 2: /Medio-Puente-W/Shunt -> GND
- C47 pad 1: /Medio-Puente-W/VB -> GND
- C47 pad 2: /Medio-Puente-W/PHASE_OUT -> /Microcontrolador/BOOT0
- C48 pad 1: GND -> +3V3
- C48 pad 2: /PA0 -> GND
- C49 pad 1: +24V -> /Microcontrolador/VCAP1
- C5 pad 1: /HSE_2 -> +3V3
- C50 pad 1: /PA1 -> +5V
- C51 pad 1: /Sensores/T1 -> +3V3
- C52 pad 1: /Sensores/T3 -> +3V3
- C53 pad 1: /Sensores/T5 -> VDDA
- C54 pad 1: /Sensores/T2 -> +5V
- C55 pad 1: /Sensores/T4 -> +3V3
- C56 pad 1: /Sensores/T6 -> +3V3
- C57 pad 1: /Sensores/12V_SENS -> +3V3
- C58 pad 1: /Sensores/24V_SENS -> Net-(U10-REFin/REFout)
- C6 pad 1: GND -> /Medio-Puente-U/VB
- C6 pad 2: /BOOT0 -> /Medio-Puente-U/PHASE_OUT
- C7 pad 1: +3V3 -> Net-(C7-Pad1)
- C8 pad 1: /VCAP1 -> Net-(D2-K)
- C8 pad 2: GND -> /Medio-Puente-U/Shunt
- C9 pad 1: +3V3 -> /Medio-Puente-U/VB
- C9 pad 2: GND -> /Medio-Puente-U/PHASE_OUT
- D1 pad 1: GND -> Net-(D1-K)
- D1 pad 2: Net-(D1-A) -> +24V
- D10 pad 1: GND -> Net-(D10-K)
- D10 pad 2: Net-(D10-A) -> /Medio-Puente-W/PHASE_OUT
- D11 pad 1: GND -> /Medio-Puente-W/VB
- D11 pad 2: +3V3 -> +12V
- D12 pad 2: Net-(D12-A2) -> /Microcontrolador/PA1
- D13 pad 2: Net-(D13-A2) -> /Protección 24V-12V/24V fused
- D14 pad 1: GND -> /Protección 24V-12V/24V fused
- D14 pad 2: Net-(D14-A2) -> +24V
- D15 pad 1: /SWSCK -> GND
- D15 pad 2: /SWDIO -> Net-(D15-A)
- D16 pad 1: /PB3 -> GND
- D16 pad 2: /PB4 -> +12V
- D17 pad 1: /PB5 -> GND
- D17 pad 2: +3V3 -> Net-(D17-A)
- D18 pad 1: GND -> /Microcontrolador/USB_R_N
- D18 pad 2: +12V -> /Microcontrolador/USB_R_P
- D19 pad 1: /I2C_SCL -> GND
- D19 pad 2: /I2C_SDA -> +5V
- D2 pad 1: /PA15 -> Net-(D2-K)
- D2 pad 2: Net-(D2-A) -> /Medio-Puente-U/PHASE_OUT
- D20 pad 1: Net-(D20-K) -> GND
- D20 pad 2: +24V -> Net-(D20-A)
- D21 pad 1: Net-(D21-K) -> /Microcontrolador/PA15
- D21 pad 2: /Medio-Puente-U/PHASE_OUT -> Net-(D21-A)
- D22 pad 1: /Medio-Puente-U/VB -> /Microcontrolador/SWSCK
- D22 pad 2: +12V -> /Microcontrolador/SWDIO
- D23 pad 2: /PB0 -> +3V3
- D24 pad 1: Net-(D24-K) -> /Microcontrolador/I2C_SDA
- D24 pad 2: +24V -> /Microcontrolador/I2C_SCL
- D25 pad 1: Net-(D25-K) -> GND
- D25 pad 2: /Medio-Puente-V/PHASE_OUT -> Net-(D25-A)
- D26 pad 1: /Medio-Puente-V/VB -> +24V
- D26 pad 2: +12V -> Net-(D26-A)
- D27 pad 1: GND -> /Microcontrolador/PB3
- D27 pad 2: /PA4 -> +3V3
- D28 pad 1: Net-(D28-K) -> /Microcontrolador/PB5
- D28 pad 2: +24V -> /Microcontrolador/PB4
- D29 pad 1: Net-(D29-K) -> GND
- D29 pad 2: /Medio-Puente-W/PHASE_OUT -> /Medio-Puente-U/PHASE_OUT
- D3 pad 1: GND -> /Medio-Puente-U/VB
- D3 pad 2: Net-(D3-A) -> +12V
- D30 pad 1: /Medio-Puente-W/VB -> GND
- D30 pad 2: +12V -> /Medio-Puente-V/PHASE_OUT
- D31 pad 2: /PA0 -> /Medio-Puente-W/PHASE_OUT
- D4 pad 2: Net-(D4-A) -> /Microcontrolador/PB1
- D5 pad 1: GND -> Net-(D5-K)
- D5 pad 2: /24V fused -> +24V
- D6 pad 1: /24V fused -> Net-(D6-K)
- D6 pad 2: +24V -> /Medio-Puente-V/PHASE_OUT
- D7 pad 1: /USB_R_N -> /Medio-Puente-V/VB
- D7 pad 2: /USB_R_P -> +12V
- D8 pad 2: /5V fused -> /Microcontrolador/PA5
- D9 pad 1: +5V -> Net-(D9-K)
- D9 pad 2: /5V fused -> +24V
- F1 pad 1: /24V in -> /Protección 24V-12V/24V in
- F1 pad 2: /24V fused -> /Protección 24V-12V/24V fused
- F3 pad 2: /5V fused -> +5V
- J1 pad 1: /24V in -> GND
- J1 pad 2: GND -> /Microcontrolador/PA9
- J10 pad 1: /Medio-Puente-V/PHASE_OUT -> +24V
- J11 pad 1: /Medio-Puente-W/PHASE_OUT -> GND
- J12 pad 1: +3V3 -> GND
- J12 pad 2: /Contactor-Control/SDA -> /ADC/CH4
- J12 pad 3: /Contactor-Control/SCL -> /ADC/CH5
- J13 pad 1: +24V -> GND
- J13 pad 2: GND -> /Microcontrolador/PA3
- J14 pad 1: /Contactor-Control/Phase -> GND
- J14 pad 2: /Contactor-Control/Neutral -> +12V
- J15 pad 1: /Contactor-Control/Neutral -> /Medio-Puente-W/PHASE_OUT
- J3 pad 1: Net-(D14-A2) -> /Medio-Puente-U/PHASE_OUT
- J4 pad 1: Net-(D12-A2) -> +24V
- J5 pad 1: Net-(D13-A2) -> GND
- J6 pad 1: Net-(D14-A2) -> GND
- J7 pad 2: GND -> /Microcontrolador/PA7
- J7 pad 3: /SWSCK -> /Microcontrolador/PA6
- J7 pad 4: /I2C_SCL -> /Microcontrolador/PA5
- J7 pad 5: /SWDIO -> /Microcontrolador/PA4
- J7 pad 6: /I2C_SDA -> +3V3
- J8 pad 2: /PB3 -> +12V
- J9 pad 1: /Medio-Puente-U/PHASE_OUT -> /Medio-Puente-V/PHASE_OUT
- L2 pad 2: Net-(Q1-D) -> Net-(Q7-D)
- Q1 pad 2: GND -> +24V
- Q1 pad 3: Net-(Q1-D) -> /Medio-Puente-U/PHASE_OUT
- Q2 pad 2: +24V -> /Medio-Puente-U/PHASE_OUT
- Q2 pad 3: /Medio-Puente-U/PHASE_OUT -> /Medio-Puente-U/Shunt
- Q3 pad 2: /Medio-Puente-U/PHASE_OUT -> +24V
- Q3 pad 3: /Medio-Puente-U/Shunt -> /Medio-Puente-V/PHASE_OUT
- Q4 pad 2: +24V -> /Medio-Puente-V/PHASE_OUT
- Q4 pad 3: /Medio-Puente-V/PHASE_OUT -> /Medio-Puente-V/Shunt
- Q5 pad 2: /Medio-Puente-V/PHASE_OUT -> +24V
- Q5 pad 3: /Medio-Puente-V/Shunt -> /Medio-Puente-W/PHASE_OUT
- Q6 pad 2: +24V -> /Medio-Puente-W/PHASE_OUT
- Q6 pad 3: /Medio-Puente-W/PHASE_OUT -> /Medio-Puente-W/Shunt
- Q7 pad 2: /Medio-Puente-W/PHASE_OUT -> GND
- Q7 pad 3: /Medio-Puente-W/Shunt -> Net-(Q7-D)
- Q9 pad 2: Net-(D32-A) -> Net-(D26-A)
- R1 pad 1: +3V3 -> /Medio-Puente-U/Shunt
- R1 pad 2: Net-(D1-A) -> GND
- R10 pad 1: /USB_N -> Net-(Q2-G)
- R10 pad 2: /USB_R_N -> Net-(U1-LO)
- R11 pad 1: /USB_P -> /ADC/CH3
- R11 pad 2: /USB_R_P -> Net-(C7-Pad1)
- R12 pad 1: /PB7 -> /Medio-Puente-U/PHASE_OUT
- R13 pad 1: GND -> /Medio-Puente-U/Shunt
- R13 pad 2: Net-(Q1-G) -> Net-(Q2-G)
- R14 pad 1: /V_DIV_3 -> /Microcontrolador/PB0
- R14 pad 2: GND -> /Medio-Puente-U/PHASE_OUT
- R15 pad 1: +5V -> GND
- R15 pad 2: Net-(R15-Pad2) -> /Microcontrolador/PB0
- R16 pad 1: Net-(R15-Pad2) -> /Medio-Puente-V/Shunt
- R16 pad 2: Net-(D10-A) -> GND
- R17 pad 1: +3V3 -> Net-(D5-K)
- R17 pad 2: /V_DIV_3 -> +24V
- R18 pad 1: GND -> Net-(C14-Pad1)
- R18 pad 2: /V_DIV_12 -> +3V3
- R19 pad 1: +12V -> Net-(R19-Pad1)
- R2 pad 1: +3V3 -> Net-(D1-K)
- R2 pad 2: Net-(D2-A) -> +24V
- R20 pad 1: Net-(R19-Pad2) -> /ADC/CH4
- R20 pad 2: Net-(R20-Pad2) -> Net-(C14-Pad1)
- R21 pad 1: /PB3 -> Net-(D6-K)
- R21 pad 2: +3V3 -> /Medio-Puente-V/PHASE_OUT
- R22 pad 1: Net-(R20-Pad2) -> Net-(R22-Pad1)
- R22 pad 2: /V_DIV_12 -> /Microcontrolador/PA5
- R23 pad 1: /PB4 -> Net-(C19-Pad1)
- R24 pad 1: /PB5 -> Net-(U3-HO)
- R24 pad 2: +3V3 -> Net-(Q3-G)
- R25 pad 1: /I2C_SCL -> Net-(Q4-G)
- R25 pad 2: +3V3 -> Net-(U3-LO)
- R26 pad 1: /I2C_SDA -> /ADC/CH5
- R26 pad 2: +3V3 -> Net-(C19-Pad1)
- R27 pad 1: /Medio-Puente-U/Shunt -> /Medio-Puente-V/PHASE_OUT
- R27 pad 2: GND -> Net-(Q3-G)
- R28 pad 1: Net-(D20-K) -> /Medio-Puente-V/Shunt
- R28 pad 2: +24V -> Net-(Q4-G)
- R29 pad 1: Net-(R29-Pad1) -> /Microcontrolador/PA4
- R29 pad 2: Net-(R29-Pad2) -> /Medio-Puente-V/PHASE_OUT
- R3 pad 1: GND -> Net-(C2-Pad1)
- R3 pad 2: /BOOT0 -> +3V3
- R30 pad 1: Net-(D21-K) -> GND
- R30 pad 2: /Medio-Puente-U/PHASE_OUT -> /Microcontrolador/PA4
- R31 pad 1: Net-(R31-Pad1) -> /Medio-Puente-W/Shunt
- R31 pad 2: /PB0 -> GND
- R32 pad 1: Net-(U5-HO) -> Net-(D9-K)
- R32 pad 2: Net-(Q2-G) -> +24V
- R33 pad 1: Net-(Q3-G) -> Net-(C26-Pad1)
- R33 pad 2: Net-(U5-LO) -> +3V3
- R34 pad 1: /Medio-Puente-U/PHASE_OUT -> Net-(R34-Pad1)
- R34 pad 2: Net-(Q2-G) -> Net-(R34-Pad2)
- R35 pad 1: /Medio-Puente-U/Shunt -> /ADC/CH6
- R35 pad 2: Net-(Q3-G) -> Net-(C26-Pad1)
- R36 pad 1: /PB1 -> Net-(D10-K)
- R36 pad 2: /Medio-Puente-U/PHASE_OUT -> /Medio-Puente-W/PHASE_OUT
- R37 pad 1: GND -> Net-(R37-Pad1)
- R37 pad 2: /PB1 -> /Microcontrolador/PA1
- R38 pad 1: /Medio-Puente-V/Shunt -> Net-(C31-Pad1)
- R38 pad 2: GND -> +3V3
- R39 pad 1: Net-(D24-K) -> Net-(U5-HO)
- R39 pad 2: +24V -> Net-(Q5-G)
- R4 pad 1: +3V3 -> Net-(R4-Pad1)
- R4 pad 2: /NRST -> Net-(R4-Pad2)
- R40 pad 1: Net-(R40-Pad1) -> Net-(Q6-G)
- R40 pad 2: Net-(R40-Pad2) -> Net-(U5-LO)
- R41 pad 1: Net-(D25-K) -> /ADC/CH7
- R41 pad 2: /Medio-Puente-V/PHASE_OUT -> Net-(C31-Pad1)
- R42 pad 1: Net-(R42-Pad1) -> /Medio-Puente-W/PHASE_OUT
- R42 pad 2: /PA4 -> Net-(Q5-G)
- R43 pad 1: Net-(U7-HO) -> /Medio-Puente-W/Shunt
- R43 pad 2: Net-(Q4-G) -> Net-(Q6-G)
- R44 pad 1: Net-(Q5-G) -> /Microcontrolador/PA0
- R44 pad 2: Net-(U7-LO) -> /Medio-Puente-W/PHASE_OUT
- R45 pad 1: /Medio-Puente-V/PHASE_OUT -> GND
- R45 pad 2: Net-(Q4-G) -> /Microcontrolador/PA0
- R46 pad 1: /Medio-Puente-V/Shunt -> +24V
- R46 pad 2: Net-(Q5-G) -> Net-(D15-A)
- R47 pad 1: /PA5 -> +24V
- R47 pad 2: /Medio-Puente-V/PHASE_OUT -> /ADC/CH0
- R48 pad 2: /PA5 -> /ADC/CH0
- R49 pad 1: /Medio-Puente-W/Shunt -> GND
- R49 pad 2: GND -> /Protección 24V-12V/V_DIV_12
- R5 pad 1: Net-(D3-A) -> /ADC/CH2
- R5 pad 2: +12V -> Net-(C2-Pad1)
- R50 pad 1: Net-(D28-K) -> +12V
- R50 pad 2: +24V -> Net-(R50-Pad2)
- R51 pad 1: Net-(R51-Pad1) -> Net-(R50-Pad2)
- R52 pad 1: Net-(D29-K) -> Net-(R51-Pad2)
- R52 pad 2: /Medio-Puente-W/PHASE_OUT -> /Protección 24V-12V/V_DIV_12
- R53 pad 1: Net-(R53-Pad1) -> +12V
- R53 pad 2: /PA0 -> Net-(D17-A)
- R54 pad 1: Net-(U9-HO) -> +12V
- R54 pad 2: Net-(Q6-G) -> Net-(D17-A)
- R55 pad 1: Net-(Q7-G) -> +12V
- R55 pad 2: Net-(U9-LO) -> /ADC/CH1
- R56 pad 1: /Medio-Puente-W/PHASE_OUT -> /ADC/CH1
- R56 pad 2: Net-(Q6-G) -> GND
- R57 pad 1: /Medio-Puente-W/Shunt -> GND
- R57 pad 2: Net-(Q7-G) -> /Microcontrolador/BOOT0
- R58 pad 1: /PA1 -> +3V3
- R58 pad 2: /Medio-Puente-W/PHASE_OUT -> /Microcontrolador/NRST
- R59 pad 1: GND -> /Microcontrolador/USB_R_N
- R59 pad 2: /PA1 -> /Microcontrolador/USB_N
- R6 pad 1: +12V -> Net-(D2-K)
- R6 pad 2: Net-(D3-A) -> /Medio-Puente-U/PHASE_OUT
- R60 pad 1: /Sensores/T1 -> /Microcontrolador/USB_R_P
- R60 pad 2: +3V3 -> /Microcontrolador/USB_P
- R61 pad 1: /Sensores/T3 -> /Microcontrolador/USB_CC2
- R61 pad 2: +3V3 -> GND
- R62 pad 1: /Sensores/T5 -> GND
- R62 pad 2: +3V3 -> /Microcontrolador/USB_CC1
- R63 pad 1: /Sensores/S1 -> +5V
- R63 pad 2: /Sensores/T1 -> Net-(R63-Pad2)
- R64 pad 1: /Sensores/S3 -> Net-(R63-Pad2)
- R64 pad 2: /Sensores/T3 -> Net-(D20-A)
- R65 pad 1: /Sensores/S5 -> +3V3
- R65 pad 2: /Sensores/T5 -> Net-(D21-A)
- R66 pad 1: /Sensores/T2 -> /Microcontrolador/PB7
- R66 pad 2: +3V3 -> Net-(Q7-G)
- R67 pad 1: /Sensores/T4 -> /Microcontrolador/V_DIV_3
- R67 pad 2: +3V3 -> GND
- R68 pad 1: /Sensores/T6 -> GND
- R68 pad 2: +3V3 -> Net-(Q7-G)
- R69 pad 1: /Sensores/S2 -> +3V3
- R69 pad 2: /Sensores/T2 -> /Microcontrolador/V_DIV_3
- R7 pad 1: +24V -> Net-(R7-Pad1)
- R7 pad 2: Net-(D4-A) -> /Microcontrolador/PB1
- R70 pad 1: /Sensores/S4 -> /Microcontrolador/I2C_SCL
- R70 pad 2: /Sensores/T4 -> +3V3
- R71 pad 1: /Sensores/S6 -> /Microcontrolador/I2C_SDA
- R71 pad 2: /Sensores/T6 -> +3V3
- R72 pad 1: /Sensores/12V_SENS -> +3V3
- R72 pad 2: +12V -> Net-(D25-A)
- R73 pad 1: /Sensores/24V_SENS -> /Microcontrolador/PA10
- R73 pad 2: +24V -> Net-(Q8-B)
- R74 pad 1: /Sensores/12V_SENS -> +24V
- R74 pad 2: GND -> Net-(Q8-C)
- R75 pad 1: GND -> /Contactor/OUT_R
- R75 pad 2: /Sensores/24V_SENS -> /Protección 24V-12V/24V in
- R76 pad 1: Net-(U11-PB1) -> /Microcontrolador/PB3
- R76 pad 2: Net-(Q8-B) -> +3V3
- R77 pad 1: +24V -> /Microcontrolador/PB4
- R77 pad 2: Net-(Q8-C) -> +3V3
- R8 pad 1: GND -> Net-(C7-Pad1)
- R8 pad 2: /USB_CC1 -> +3V3
- R9 pad 1: GND -> Net-(U1-HO)
- R9 pad 2: /USB_CC2 -> Net-(Q1-G)
- SW1 pad 2: /BOOT0 -> /Microcontrolador/BOOT0
- SW2 pad 2: /NRST -> /Microcontrolador/NRST
- TH1 pad 1: /Sensores/T1 -> Net-(C2-Pad1)
- TH2 pad 1: /Sensores/T3 -> Net-(C7-Pad1)
- TH3 pad 1: /Sensores/T5 -> Net-(C14-Pad1)
- TH4 pad 1: /Sensores/T2 -> Net-(C19-Pad1)
- TH5 pad 1: /Sensores/T4 -> Net-(C26-Pad1)
- TH6 pad 1: /Sensores/T6 -> Net-(C31-Pad1)
- U1 pad 1: unconnected-(U1-VBAT-Pad1) -> +12V
- U1 pad 2: /PC13 -> /Microcontrolador/PA9
- U1 pad 3: /LSE_1 -> /Microcontrolador/PA8
- U1 pad 4: /LSE_2 -> GND
- U1 pad 5: /HSE_1 -> Net-(U1-LO)
- U1 pad 6: /HSE_2 -> /Medio-Puente-U/PHASE_OUT
- U1 pad 7: /NRST -> Net-(U1-HO)
- U1 pad 8: GND -> /Medio-Puente-U/VB
- U10 pad 1: GND -> /ADC/CH0
- U10 pad 2: Net-(R51-Pad1) -> /ADC/CH1
- U10 pad 3: Net-(R51-Pad2) -> /ADC/CH2
- U10 pad 4: /Medio-Puente-W/Shunt -> /ADC/CH3
- U10 pad 5: GND -> /ADC/CH4
- U10 pad 6: GND -> /ADC/CH5
- U10 pad 7: Net-(R53-Pad1) -> /ADC/CH6
- U10 pad 8: +3V3 -> /ADC/CH7
- U2 pad 1: /V_DIV_3 -> GND
- U2 pad 2: +3V3 -> Net-(R4-Pad1)
- U2 pad 3: +5V -> Net-(R4-Pad2)
- U3 pad 1: /Sensores/24V_SENS -> +12V
- U3 pad 2: /Sensores/12V_SENS -> /Microcontrolador/PA7
- U3 pad 3: /Sensores/S1 -> /Microcontrolador/PA6
- U3 pad 4: /Sensores/S2 -> GND
- U3 pad 5: /Sensores/S3 -> Net-(U3-LO)
- U3 pad 6: /Sensores/S4 -> /Medio-Puente-V/PHASE_OUT
- U3 pad 7: /Sensores/S5 -> Net-(U3-HO)
- U3 pad 8: /Sensores/S6 -> /Medio-Puente-V/VB
- U4 pad 1: /V_DIV_12 -> GND
- U4 pad 2: +12V -> Net-(R19-Pad1)
- U4 pad 3: +24V -> Net-(R19-Pad2)
- U5 pad 2: /PA9 -> /Microcontrolador/PA3
- U5 pad 3: /PA8 -> /Microcontrolador/PA2
- U5 pad 6: /Medio-Puente-U/PHASE_OUT -> /Medio-Puente-W/PHASE_OUT
- U5 pad 8: /Medio-Puente-U/VB -> /Medio-Puente-W/VB
- U6 pad 2: Net-(R29-Pad1) -> Net-(R34-Pad1)
- U6 pad 3: Net-(R29-Pad2) -> Net-(R34-Pad2)
- U6 pad 4: /Medio-Puente-U/Shunt -> /Medio-Puente-W/Shunt
- U6 pad 7: Net-(R31-Pad1) -> Net-(R37-Pad1)
- U7 pad 1: +12V -> /Protección 24V-12V/V_DIV_12
- U7 pad 2: /PA7 -> +12V
- U7 pad 3: /PA6 -> +24V
- U8 pad 1: GND -> unconnected-(U8-VBAT-Pad1)
- U8 pad 2: Net-(R40-Pad1) -> /Microcontrolador/PC13
- U8 pad 3: Net-(R40-Pad2) -> /Microcontrolador/LSE_1
- U8 pad 4: /Medio-Puente-V/Shunt -> /Microcontrolador/LSE_2
- U8 pad 5: GND -> /Microcontrolador/HSE_1
- U8 pad 6: GND -> /Microcontrolador/HSE_2
- U8 pad 7: Net-(R42-Pad1) -> /Microcontrolador/NRST
- U8 pad 8: +3V3 -> GND
- U9 pad 1: +12V -> /Microcontrolador/V_DIV_3
- U9 pad 2: /PA3 -> +3V3
- U9 pad 3: /PA2 -> +5V
- Y1 pad 1: /HSE_1 -> /Microcontrolador/HSE_1
- Y1 pad 3: /HSE_2 -> /Microcontrolador/HSE_2
- Y2 pad 1: /LSE_1 -> /Microcontrolador/LSE_1
- Y2 pad 2: /LSE_2 -> /Microcontrolador/LSE_2
Routing:
- net +12V: track 203.9 -> 47.3 mm, vias 3 -> 0
- net /PB7: track 107.1 -> 0.00 mm, vias 2 -> 0
- net /I2C_SDA: track 104.6 -> 0.00 mm, vias 2 -> 0
- net /Sensores/24V_SENS: track 101.0 -> 0.00 mm, vias 2 -> 0
- net /Sensores/12V_SENS: track 99.1 -> 0.00 mm, vias 2 -> 0
- net /I2C_SCL: track 98.4 -> 0.00 mm, vias 2 -> 0
- net +24V: track 177.8 -> 87.7 mm, vias 2 -> 93
- net /ADC/CH4: track 0.00 -> 79.2 mm
- net /ADC/CH2: track 0.00 -> 77.6 mm
- net /ADC/CH6: track 0.00 -> 77.5 mm
- net GND: track 214.8 -> 145.4 mm, vias 751 -> 232
- net /PB1: track 65.5 -> 0.00 mm
- net /PA1: track 63.2 -> 0.00 mm
- net /PA9: track 62.3 -> 0.00 mm
- net /PA0: track 62.3 -> 0.00 mm
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- added copper zone on F.Cu, net +12V
- added copper zone on F.Cu, net +24V
- added copper zone on F.Cu, net /Contactor/OUT_R
- added copper zone on B.Cu, net /Medio-Puente-U/PHASE_OUT
- added copper zone on F.Cu, net /Medio-Puente-U/PHASE_OUT
- added copper zone on B.Cu, net /Medio-Puente-U/Shunt
- added copper zone on B.Cu, net /Medio-Puente-V/PHASE_OUT
- added copper zone on F.Cu, net /Medio-Puente-V/PHASE_OUT
- added copper zone on B.Cu, net /Medio-Puente-V/Shunt
- added copper zone on B.Cu, net /Medio-Puente-W/PHASE_OUT
- added copper zone on F.Cu, net /Medio-Puente-W/PHASE_OUT
- added copper zone on B.Cu, net /Medio-Puente-W/Shunt
- added copper zone on F.Cu, net /Protección 24V-12V/24V fused
- added copper zone on B.Cu, net /Protección 24V-12V/24V in
- added copper zone on F.Cu, net /Protección 24V-12V/24V in
- removed copper zone on F.Cu, net /24V fused
- removed copper zone on In1.Cu, net /24V fused
- removed copper zone on In2.Cu, net /24V fused
- removed copper zone on B.Cu, net /24V in
- removed copper zone on F.Cu, net /24V in
- removed copper zone on In1.Cu, net /24V in
- removed copper zone on In2.Cu, net /24V in
- removed copper zone on In1.Cu, net GND
- removed copper zone on In2.Cu, net GND
Other:
- board size 155 x 111.3 mm -> 217.3 x 252.1 mm
- copper layers 4 -> 2
- board text added: "12 V"
- board text added: "3.3 V"
- board text added: "5 V"
- board text added: "BOOT0"
- board text added: "Board: 70 x 30 mm Holes: 60 x 20 mm"
- board text added: "CONTACTOR"
- board text added: "FAN"
- board text added: "GND 24Vs 12Vs"
- board text added: "GND SCL SDA"
- board text added: "GND TUH TUL TVH TVL TWH TWL 3V3"
- board text added: "HALF BRIDGE"
- board text added: "HALL SENS."
- board text added: "I MAX: 39 Ar V MAX: 36 V"
- board text added: "I^{2}C"
- board text added: "MCU"
- board text added: "POWER BOARD"
- board text added: "U PHASE"
- board text added: "V PHASE"
- board text added: "W PHASE"
- board text removed: "+"
- board text removed: "+24V DC"
- board text removed: "-"
- board text removed: "230V AC"
- board text removed: "24V MAX"
- board text removed: "ADS7830"
- board text removed: "BOOT"
- board text removed: "Botones"
- board text removed: "Contactor Coil"
- board text removed: "DANGER: MAINS VOLTAGE RISK OF ELECTROCUTION"
- board text removed: "HB-9500-2P"
- board text removed: "Medio Puente U"
- board text removed: "Medio Puente V"
- board text removed: "Medio Puente W"
- board text removed: "Microcontrolador"
- board text removed: "N"
- board text removed: "P"
- board text removed: "Protec. 24V"
- board text removed: "Protección 5V"
- board text removed: "Puerto USB-C"
- board text removed: "Reg. 3.3V"
- board text removed: "Regulador 12V"
- board text removed: "STM32F411CEUx"
- board text removed: "Salida motor"
- board text removed: "Sensores 12-24V"
- board text removed: "Sensores Hall"
- board text removed: "Sensores de Temperatura y ADC"
- board text removed: "USER"
- board text removed: "V SIO SCK G V SDA SCL G"
- board text removed: "V2"
- board text removed: "Ventilador"
- board text removed: "github.com/AdriTeixeHax"
