File: RTSpeed-KiCad/Sensores.kicad_sch (KiCad schematic)
At the start: 30 parts

Commit message: PCB redesign (not final)
Parts:
- removed C51, C52, C53, C54, C55, C56: 100n, Capacitor_SMD:C_0603_1608Metric, symbol Device:C
- removed R60, R61, R62, R66, R67, R68: 10k 1%, Resistor_SMD:R_0603_1608Metric, symbol Device:R_US
- removed R63, R64, R65, R69, R70, R71: 22R, Resistor_SMD:R_0603_1608Metric, symbol Device:R_US
- removed TH1, TH2, TH3, TH4, TH5, TH6: 10k, TFG-Brushless-ESC:temp sensor, symbol Device:Thermistor_NTC
Other:
- note removed: "Sensores de temperatura (1 por MOSFET)"
