File: RTSpeed-KiCad/contactorControl.kicad_sch (KiCad schematic)
At the start: 11 parts, among them J12 I^{2}C, J13 24V DC, J14 230V AC, J15 Contactor Coil, K1 Relay 24VDC, Q8 2N2222, Q9 IRFB4321, U11 ATtiny85-20P

Commit message: Contactor control pcb
Parts:
- added H5, H6, H7, H9: M3, MountingHole:MountingHole_3.2mm_M3, symbol Mechanical:MountingHole
- K1: footprint Relay_THT:Relay_SPDT_HsinDa_Y14 -> ESC-TFG-KiCad:OMRON G2R-1
Connections:
- net +24V: now also K1.1; no longer K1.4
- net Cont Ctrl: now also K1.4; no longer K1.5, K1.6
- net Phase: now also K1.3; no longer K1.1
- net at D32.2 (A), Q9.2 (D): now also K1.5; no longer K1.3
Other:
- note added: "Tornillos"

Commit message: PCB redesign (not final)
Parts:
- Q8: footprint Package_TO_SOT_THT:TO-92 -> Package_TO_SOT_THT:TO-92_Inline
Connections:
- net at U11.3 (XTAL2/PB4): now also R76.1
- net at U11.6 (PB1): no longer R76.1
Changed lines of the file:
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@@
+	)
+	(no_connect
+		(at 58.42 60.96)
 	)
 	(no_connect
@@
 	)
 	(no_connect
-		(at 58.42 68.58)
-	)
-	(no_connect
 		(at 58.42 71.12)
 	)
@@
 	(wire
 		(pts
+			(xy 76.2 60.96) (xy 77.47 60.96)
+		)
+		(stroke
+			(width 0)
+			(type default)
+		)
+	)
+	(wire
+		(pts
 			(xy 58.42 63.5) (xy 72.39 63.5)
 		)
@@
 	(wire
 		(pts
-			(xy 58.42 60.96) (xy 77.47 60.96)
+			(xy 76.2 68.58) (xy 58.42 68.58)
 		)
 		(stroke
@@
 		(pts
 			(xy 115.57 29.21) (xy 115.57 30.48)
+		)
+		(stroke
+			(width 0)
+			(type default)
+		)
+	)
+	(wire
+		(pts
+			(xy 76.2 60.96) (xy 76.2 68.58)
 		)
 		(stroke
@@
 			)
 		)
-		(property "Footprint" "Package_TO_SOT_THT:TO-92"
+		(property "Footprint" "Package_TO_SOT_THT:TO-92_Inline"
 			(at 153.67 60.96 0)
 			(effects
